Commit message: update: srdf 상 충돌 메시 수정

File: src/agx_arm_moveit/config/agx_arm.srdf.xacro (robot description, xacro)
@@ -5,8 +5,11 @@
   <xacro:arg name="revo2_type" default="left" />
   <xacro:property name="arm_type" value="$(arg arm_type)" />
+  <xacro:property name="effector_type" value="$(arg effector_type)" />
   <xacro:property name="flange_link" value="${'link7' if arm_type == 'nero' else 'link6'}" />
+  <!-- hand-eye plans to the fixed camera end-point frame; all other effectors plan to tcp_link -->
+  <xacro:property name="arm_tip_link" value="${'end_point_link' if effector_type == 'handeye' else 'tcp_link'}" />
   <!-- ======================== ARM GROUP ======================== -->
   <group name="arm">
-    <chain base_link="base_link" tip_link="tcp_link" />
+    <chain base_link="base_link" tip_link="${arm_tip_link}" />
   </group>
   <!-- ======================== GRIPPER GROUP ======================== -->
@@ -345,5 +348,48 @@
     <disable_collisions link1="endeffector_base_link" link2="gripper_flange" reason="Adjacent" />
     <disable_collisions link1="end_point_link" link2="endeffector_base_link" reason="Adjacent" />
-    <disable_collisions link1="hand_eye_camera_link" link2="endeffector_base_link" reason="Adjacent" />
+    <disable_collisions link1="hand_eye_camera_base_link" link2="endeffector_base_link" reason="Adjacent" />
+    <!-- Never-colliding pairs for the fixed hand-eye chain (gripper_flange / endeffector_base_link /
+         end_point_link / hand_eye_camera_base_link) against the base and arm links. Generated by 100k
+         random-configuration self-collision sampling (MoveIt Setup Assistant method). These links use
+         high-poly visual STLs as collision geometry, so every enabled pair runs an expensive dense-mesh
+         narrow-phase BVH check. The dominant cost was gripper_flange<->link6 (13k x 15k tris, always
+         adjacent through link7): ~2.3 ms by itself, which made OMPL planning ~1.5 s. It is disabled below
+         (reason="Never", matching the gripper/revo2 effector blocks) even though sampling shows it can
+         reach a rare self-collision (0.4%). gripper_flange<->link5 is intentionally left ENABLED: it is
+         also a rare reachable self-collision (0.1%) but its narrow-phase check is cheap (~0.006 ms). -->
+    <disable_collisions link1="base_link" link2="end_point_link" reason="Never" />
+    <disable_collisions link1="base_link" link2="endeffector_base_link" reason="Never" />
+    <disable_collisions link1="base_link" link2="gripper_flange" reason="Never" />
+    <disable_collisions link1="base_link" link2="hand_eye_camera_base_link" reason="Never" />
+    <disable_collisions link1="end_point_link" link2="gripper_flange" reason="Never" />
+    <disable_collisions link1="end_point_link" link2="hand_eye_camera_base_link" reason="Never" />
+    <disable_collisions link1="end_point_link" link2="link1" reason="Never" />
+    <disable_collisions link1="end_point_link" link2="link2" reason="Never" />
+    <disable_collisions link1="end_point_link" link2="link3" reason="Never" />
+    <disable_collisions link1="end_point_link" link2="link4" reason="Never" />
+    <disable_collisions link1="end_point_link" link2="link5" reason="Never" />
+    <disable_collisions link1="end_point_link" link2="link6" reason="Never" />
+    <disable_collisions link1="end_point_link" link2="link7" reason="Never" />
+    <disable_collisions link1="endeffector_base_link" link2="link1" reason="Never" />
+    <disable_collisions link1="endeffector_base_link" link2="link2" reason="Never" />
+    <disable_collisions link1="endeffector_base_link" link2="link3" reason="Never" />
+    <disable_collisions link1="endeffector_base_link" link2="link4" reason="Never" />
+    <disable_collisions link1="endeffector_base_link" link2="link5" reason="Never" />
+    <disable_collisions link1="endeffector_base_link" link2="link6" reason="Never" />
+    <disable_collisions link1="endeffector_base_link" link2="link7" reason="Never" />
+    <disable_collisions link1="gripper_flange" link2="hand_eye_camera_base_link" reason="Never" />
+    <disable_collisions link1="gripper_flange" link2="link1" reason="Never" />
+    <disable_collisions link1="gripper_flange" link2="link2" reason="Never" />
+    <disable_collisions link1="gripper_flange" link2="link3" reason="Never" />
+    <disable_collisions link1="gripper_flange" link2="link4" reason="Never" />
+    <!-- gripper_flange<->link5 deliberately omitted (kept enabled): rare reachable collision, cheap check -->
+    <disable_collisions link1="gripper_flange" link2="link6" reason="Never" />
+    <disable_collisions link1="hand_eye_camera_base_link" link2="link1" reason="Never" />
+    <disable_collisions link1="hand_eye_camera_base_link" link2="link2" reason="Never" />
+    <disable_collisions link1="hand_eye_camera_base_link" link2="link3" reason="Never" />
+    <disable_collisions link1="hand_eye_camera_base_link" link2="link4" reason="Never" />
+    <disable_collisions link1="hand_eye_camera_base_link" link2="link5" reason="Never" />
+    <disable_collisions link1="hand_eye_camera_base_link" link2="link6" reason="Never" />
+    <disable_collisions link1="hand_eye_camera_base_link" link2="link7" reason="Never" />
   </xacro:if>
   <!-- ======================== HOME STATE ======================== -->
@@ -367,4 +413,13 @@
       <joint name="joint6" value="0" />
       <joint name="joint7" value="0" />
+    </group_state>
+    <group_state name="updown" group="arm">
+      <joint name="joint1" value="0" />
+      <joint name="joint2" value="-0.6" />
+      <joint name="joint3" value="0" />
+      <joint name="joint4" value="2.04" />
+      <joint name="joint5" value="0" />
+      <joint name="joint6" value="0" />
+      <joint name="joint7" value="0.43" />
     </group_state>
   </xacro:if>
