Commit message: feat: 실물 Nero를 topic 기반 ros2_control HW로 편입 (+ nero_hardware_interface 브리지, control_gate 제거)
- agx_arm.ros2_control.xacro: mock_components/GenericSystem -> joint_state_topic_hardware_interface/JointStateTopicSystem (명령 control/joint_states, 상태 feedback/joint_states). arm 조인트 effort state_interface 추가.
- nero_hardware_interface.py(신규): ROS1 innfos_node 역할 브리지. control/joint_states 구독->Nero move_js, 실측->feedback/joint_states 발행. 1단계 최소(drag/guard 없음).
- nero_moveit.launch.py(신규): 실물 Nero+handeye MoveIt 단일 실행. control_gate 없음, broadcaster /joint_states, spawn 순서 JSB->arm_controller, start_interface 인자.
- nero_interface.launch.py(신규): 브리지 단독 실행.
- ros2_controllers_nero.yaml: nero+handeye만(gripper/hand 제거), update_rate 100.
- package.xml/setup.py: 의존성·엔트리 추가.

Co-Authored-By: Claude Opus 4.8 (1M context) <noreply@anthropic.com>

File: src/agx_arm_moveit/config/agx_arm.ros2_control.xacro (robot description, xacro)
@@ -5,88 +5,55 @@
     <ros2_control name="${name}" type="system">
       <hardware>
-        <plugin>mock_components/GenericSystem</plugin>
+        <!-- 항상 실물 팔: JTC 명령을 control/joint_states로 발행하고, 실측을
+             feedback/joint_states에서 구독해 상태 인터페이스에 반영한다.
+             nero_hardware_interface.py(= ROS1 innfos_node 역할)가 양 토픽 ↔ Nero 브리지. -->
+        <plugin>joint_state_topic_hardware_interface/JointStateTopicSystem</plugin>
+        <param name="joint_commands_topic">control/joint_states</param>
+        <param name="joint_states_topic">feedback/joint_states</param>
+        <param name="sum_wrapped_joint_states">false</param>
       </hardware>
       <joint name="joint1">
         <command_interface name="position" />
-        <state_interface name="position">
-          <param name="initial_value">${initial_positions['joint1']}</param>
-        </state_interface>
+        <state_interface name="position" />
         <state_interface name="velocity" />
+        <state_interface name="effort" />
       </joint>
       <joint name="joint2">
         <command_interface name="position" />
-        <state_interface name="position">
-          <param name="initial_value">${initial_positions['joint2']}</param>
-        </state_interface>
+        <state_interface name="position" />
         <state_interface name="velocity" />
+        <state_interface name="effort" />
       </joint>
       <joint name="joint3">
         <command_interface name="position" />
-        <state_interface name="position">
-          <param name="initial_value">${initial_positions['joint3']}</param>
-        </state_interface>
+        <state_interface name="position" />
         <state_interface name="velocity" />
+        <state_interface name="effort" />
       </joint>
       <joint name="joint4">
         <command_interface name="position" />
-        <state_interface name="position">
-          <param name="initial_value">${initial_positions['joint4']}</param>
-        </state_interface>
+        <state_interface name="position" />
         <state_interface name="velocity" />
+        <state_interface name="effort" />
       </joint>
       <joint name="joint5">
         <command_interface name="position" />
-        <state_interface name="position">
-          <param name="initial_value">${initial_positions['joint5']}</param>
-        </state_interface>
+        <state_interface name="position" />
         <state_interface name="velocity" />
+        <state_interface name="effort" />
       </joint>
       <joint name="joint6">
         <command_interface name="position" />
-        <state_interface name="position">
-          <param name="initial_value">${initial_positions['joint6']}</param>
-        </state_interface>
+        <state_interface name="position" />
         <state_interface name="velocity" />
+        <state_interface name="effort" />
       </joint>
       <xacro:if value="${arm_type == 'nero'}">
         <joint name="joint7">
           <command_interface name="position" />
-          <state_interface name="position">
-            <param name="initial_value">${initial_positions['joint7']}</param>
-          </state_interface>
+          <state_interface name="position" />
           <state_interface name="velocity" />
+          <state_interface name="effort" />
         </joint>
-      </xacro:if>
-      <xacro:if value="${effector_type == 'agx_gripper'}">
-        <joint name="gripper_joint1">
-          <command_interface name="position" />
-          <state_interface name="position">
-            <param name="initial_value">${initial_positions['gripper_joint1']}</param>
-          </state_interface>
-          <state_interface name="velocity" />
-        </joint>
-        <joint name="gripper_joint2">
-          <command_interface name="position" />
-          <state_interface name="position">
-            <param name="initial_value">${initial_positions['gripper_joint2']}</param>
-          </state_interface>
-          <state_interface name="velocity" />
-        </joint>
-      </xacro:if>
-      <xacro:if value="${effector_type == 'revo2' and revo2_type == 'left'}">
-        <joint name="left_thumb_metacarpal_joint"><command_interface name="position" /><state_interface name="position"><param name="initial_value">${initial_positions['left_thumb_metacarpal_joint']}</param></state_interface><state_interface name="velocity" /></joint>
-        <joint name="left_thumb_proximal_joint"><command_interface name="position" /><state_interface name="position"><param name="initial_value">${initial_positions['left_thumb_proximal_joint']}</param></state_interface><state_interface name="velocity" /></joint>
-        <joint name="left_index_proximal_joint"><command_interface name="position" /><state_interface name="position"><param name="initial_value">${initial_positions['left_index_proximal_joint']}</param></state_interface><state_interface name="velocity" /></joint>
-        <joint name="left_middle_proximal_joint"><command_interface name="position" /><state_interface name="position"><param name="initial_value">${initial_positions['left_middle_proximal_joint']}</param></state_interface><state_interface name="velocity" /></joint>
-        <joint name="left_ring_proximal_joint"><command_interface name="position" /><state_interface name="position"><param name="initial_value">${initial_positions['left_ring_proximal_joint']}</param></state_interface><state_interface name="velocity" /></joint>
-        <joint name="left_pinky_proximal_joint"><command_interface name="position" /><state_interface name="position"><param name="initial_value">${initial_positions['left_pinky_proximal_joint']}</param></state_interface><state_interface name="velocity" /></joint>
-      </xacro:if>
-      <xacro:if value="${effector_type == 'revo2' and revo2_type == 'right'}">
-        <joint name="right_thumb_metacarpal_joint"><command_interface name="position" /><state_interface name="position"><param name="initial_value">${initial_positions['right_thumb_metacarpal_joint']}</param></state_interface><state_interface name="velocity" /></joint>
-        <joint name="right_thumb_proximal_joint"><command_interface name="position" /><state_interface name="position"><param name="initial_value">${initial_positions['right_thumb_proximal_joint']}</param></state_interface><state_interface name="velocity" /></joint>
-        <joint name="right_index_proximal_joint"><command_interface name="position" /><state_interface name="position"><param name="initial_value">${initial_positions['right_index_proximal_joint']}</param></state_interface><state_interface name="velocity" /></joint>
-        <joint name="right_middle_proximal_joint"><command_interface name="position" /><state_interface name="position"><param name="initial_value">${initial_positions['right_middle_proximal_joint']}</param></state_interface><state_interface name="velocity" /></joint>
-        <joint name="right_ring_proximal_joint"><command_interface name="position" /><state_interface name="position"><param name="initial_value">${initial_positions['right_ring_proximal_joint']}</param></state_interface><state_interface name="velocity" /></joint>
-        <joint name="right_pinky_proximal_joint"><command_interface name="position" /><state_interface name="position"><param name="initial_value">${initial_positions['right_pinky_proximal_joint']}</param></state_interface><state_interface name="velocity" /></joint>
       </xacro:if>
     </ros2_control>
